Commit message: Improvements in end-effectors

File: sr_moveit_hand_config/config/shadowhand.srdf.xacro (robot description, xacro)
@@ -129,5 +129,5 @@
    <!--END EFFECTOR: Purpose: Represent information about an end effector.-->
    <xacro:macro name="finger_ee" params="prefix link_prefix finger_name hand_name" >
-    <end_effector name="${prefix}${link_prefix}tip_ee" parent_link="${prefix}palm" group="${prefix}${finger_name}" parent_group="${prefix}palm" />
+    <end_effector name="${prefix}${link_prefix}tip_ee" parent_link="${prefix}palm" group="${prefix}${finger_name}" parent_group="${prefix}wrist" />
    </xacro:macro>
   <!--VIRTUAL JOINT: Purpose: this element defines a virtual joint between a robot link and an external frame of reference (considered fixed with respect to the robot)-->
@@ -210,4 +210,5 @@
     </xacro:unless>
     <disable_collisions link1="${prefix}forearm" link2="${prefix}palm" reason="Never" />
+    <disable_collisions link1="${prefix}palm" link2="${prefix}manipulator" reason="Never" />
   </xacro:macro>
   <!-- finger to other finger with a finger in between -->

File: sr_moveit_hand_config/config/shadowhands_prefix.srdf.xacro (robot description, xacro)
@@ -41,9 +41,9 @@
     </group>
   </xacro:unless>
-  <group name="$(arg prefix)palm">
-    <chain base_link="$(arg prefix)forearm" tip_link="$(arg prefix)palm" />
+  <group name="$(arg prefix)forearm">
+    <link name="$(arg prefix)forearm" />
   </group>
-  <group name="$(arg prefix)forearm">
-    <chain base_link="$(arg prefix)forearm" tip_link="$(arg prefix)wrist" />
+  <group name="$(arg prefix)manipulator">
+    <chain base_link="$(arg prefix)forearm" tip_link="$(arg prefix)manipulator" />
   </group>
   <!-- single finger groups -->
@@ -300,6 +300,6 @@
     <end_effector group="$(arg prefix)wrist" name="$(arg prefix)wrist_ee" parent_link="$(arg prefix)forearm" parent_group="$(arg prefix)forearm"/>
   </xacro:unless>
-  <end_effector group="$(arg prefix)fingers" name="$(arg prefix)palm_ee" parent_group="$(arg prefix)palm" parent_link="$(arg prefix)palm"/>
-  <xacro:virtual_joints prefix="$(arg prefix)" />
+  <end_effector group="$(arg prefix)fingers" name="$(arg prefix)palm_ee" parent_group="$(arg prefix)wrist" parent_link="$(arg prefix)palm"/>
+  <end_effector group="$(arg prefix)fingers" name="$(arg prefix)manipulator_ee" parent_group="$(arg prefix)manipulator" parent_link="$(arg prefix)manipulator"/>
   <!--DISABLE COLLISIONS: By default it is assumed that any link of the robot could potentially come into collision with any other link in the robot. This tag disables collision checking between a specified pair of links. -->
   <xacro:hand_collisions prefix="$(arg prefix)" />
